File: wii-pmod-adapter.kicad_sch (KiCad schematic)
At the start: 22 parts, among them J1 PMOD0, J2 PMOD1, J3 PWR, J4 DATA, J5 CLK, J6 MISC

Commit message: Early layout
Parts:
- removed J1: PMOD0, symbol Connector_Generic:Conn_02x06_Row_Letter_First
- removed J2: PMOD1, symbol Connector_Generic:Conn_02x06_Row_Letter_First
- added J1, J2: Conn_02x06_Odd_Even, Connector_PinHeader_2.54mm:PinHeader_2x06_P2.54mm_Vertical, symbol Connector_Generic:Conn_02x06_Odd_Even
- D1, D17, D18, D19, D2, D20, D21, D22, D23, D24, D3, D4, D5, D6, D7, D8: footprint (none) -> Diode_SMD:D_SOD-123
- J3, J5: footprint (none) -> Connector_JST:JST_PH_B2B-PH-K_1x02_P2.00mm_Vertical
- J4: footprint (none) -> Connector_JST:JST_PH_B8B-PH-K_1x08_P2.00mm_Vertical
- J6: footprint (none) -> Connector_JST:JST_PH_B6B-PH-K_1x06_P2.00mm_Vertical
Connections:
- net +3V3: now also J1.1 (Pin_1), J1.2 (Pin_2), J2.1 (Pin_1), J2.2 (Pin_2)
- net GND: now also J1.3 (Pin_3), J1.4 (Pin_4), J2.3 (Pin_3), J2.4 (Pin_4)
- net IO0: now also J1.5 (Pin_5)
- net IO1: now also J1.6 (Pin_6)
- net IO10: now also J2.7 (Pin_7)
- net IO11: now also J2.8 (Pin_8)
- net IO12: now also J2.9 (Pin_9)
- net IO13: now also J2.10 (Pin_10)
- net IO14: now also J2.11 (Pin_11)
- net IO15: now also J2.12 (Pin_12)
- net IO2: now also J1.7 (Pin_7)
- net IO3: now also J1.8 (Pin_8)
- net IO4: now also J1.9 (Pin_9)
- net IO5: now also J1.10 (Pin_10)
- net IO6: now also J1.11 (Pin_11)
- net IO7: now also J1.12 (Pin_12)
- net IO8: now also J2.5 (Pin_5)
- net IO9: now also J2.6 (Pin_6)
Changed lines of the file:
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@@
       (effects (font (size 1.27 1.27)) hide)
     )
-    (property "Footprint" "" (at 163.83 22.86 0)
+    (property "Footprint" "Diode_SMD:D_SOD-123" (at 163.83 22.86 0)
       (effects (font (size 1.27 1.27)) hide)
     )
@@
     )
   )
-  (symbol (lib_id "Connector_Generic:Conn_02x06_Row_Letter_First") (at 85.09 57.15 0) (unit 1)
-    (in_bom yes) (on_board yes) (dnp no) (fields_autoplaced)
-    (property "Reference" "J1" (at 86.36 45.72 0)
-      (effects (font (size 1.27 1.27)))
-    )
-    (property "Value" "PMOD0" (at 86.36 48.26 0)
-      (effects (font (size 1.27 1.27)))
-    )
-    (property "Footprint" "" (at 85.09 57.15 0)
-      (effects (font (size 1.27 1.27)) hide)
-    )
-    (property "Datasheet" "~" (at 85.09 57.15 0)
-      (effects (font (size 1.27 1.27)) hide)
-    )
-    (pin "a1")
-    (pin "a2")
-    (pin "a3")
-    (pin "a4")
-    (pin "a5")
-    (pin "a6")
-    (pin "b1")
-    (pin "b2")
-    (pin "b3")
-    (pin "b4")
-    (pin "b5")
-    (pin "b6")
-    (instances
-      (project "wii-pmod-adapter"
-        (path "/3e768cc3-1b06-47e6-92bc-2e81f82d9573"
-          (reference "J1") (unit 1)
-        )
-      )
-    )
-  )
   (symbol (lib_id "Device:D_Schottky") (at 163.83 49.53 180) (unit 1)
     (in_bom yes) (on_board yes) (dnp no)
@@
       (effects (font (size 1.27 1.27)) hide)
     )
-    (property "Footprint" "" (at 163.83 49.53 0)
+    (property "Footprint" "Diode_SMD:D_SOD-123" (at 163.83 49.53 0)
       (effects (font (size 1.27 1.27)) hide)
     )
@@
       (effects (font (size 1.27 1.27)) hide)
     )
-    (property "Footprint" "" (at 163.83 45.72 0)
+    (property "Footprint" "Diode_SMD:D_SOD-123" (at 163.83 45.72 0)
       (effects (font (size 1.27 1.27)) hide)
     )
@@
       (effects (font (size 1.27 1.27)) hide)
     )
-    (property "Footprint" "" (at 163.83 76.2 0)
+    (property "Footprint" "Diode_SMD:D_SOD-123" (at 163.83 76.2 0)
       (effects (font (size 1.27 1.27)) hide)
     )
@@
       (effects (font (size 1.27 1.27)))
     )
-    (property "Footprint" "" (at 151.13 80.01 0)
+    (property "Footprint" "Connector_JST:JST_PH_B6B-PH-K_1x06_P2.00mm_Vertical" (at 151.13 80.01 0)
       (effects (font (size 1.27 1.27)) hide)
     )
@@
       (effects (font (size 1.27 1.27)) hide)
     )
-    (property "Footprint" "" (at 163.83 41.91 0)
+    (property "Footprint" "Diode_SMD:D_SOD-123" (at 163.83 41.91 0)
       (effects (font (size 1.27 1.27)) hide)
     )
@@
       (effects (font (size 1.27 1.27)))
     )
-    (property "Footprint" "" (at 151.13 34.29 0)
+    (property "Footprint" "Connector_JST:JST_PH_B8B-PH-K_1x08_P2.00mm_Vertical" (at 151.13 34.29 0)
       (effects (font (size 1.27 1.27)) hide)
     )
@@
       (effects (font (size 1.27 1.27)) hide)
     )
-    (property "Footprint" "" (at 163.83 72.39 0)
+    (property "Footprint" "Diode_SMD:D_SOD-123" (at 163.83 72.39 0)
       (effects (font (size 1.27 1.27)) hide)
     )
@@
       (effects (font (size 1.27 1.27)))
     )
-    (property "Footprint" "" (at 151.13 59.69 0)
+    (property "Footprint" "Connector_JST:JST_PH_B2B-PH-K_1x02_P2.00mm_Vertical" (at 151.13 59.69 0)
       (effects (font (size 1.27 1.27)) hide)
     )
@@
       (effects (font (size 1.27 1.27)) hide)
     )
-    (property "Footprint" "" (at 163.83 87.63 0)
+    (property "Footprint" "Diode_SMD:D_SOD-123" (at 163.83 87.63 0)
       (effects (font (size 1.27 1.27)) hide)
     )
@@
       (effects (font (size 1.27 1.27)) hide)
     )
-    (property "Footprint" "" (at 163.83 59.69 0)
+    (property "Footprint" "Diode_SMD:D_SOD-123" (at 163.83 59.69 0)
       (effects (font (size 1.27 1.27)) hide)
     )
@@
     )
   )
+  (symbol (lib_id "Connector_Generic:Conn_02x06_Odd_Even") (at 85.09 57.15 0) (unit 1)
+    (in_bom yes) (on_board yes) (dnp no) (fields_autoplaced)
+    (property "Reference" "J1" (at 86.36 45.72 0)
+      (effects (font (size 1.27 1.27)))
+    )
+    (property "Value" "Conn_02x06_Odd_Even" (at 86.36 48.26 0)
+      (effects (font (size 1.27 1.27)))
+    )
+    (property "Footprint" "Connector_PinHeader_2.54mm:PinHeader_2x06_P2.54mm_Vertical" (at 85.09 57.15 0)
+      (effects (font (size 1.27 1.27)) hide)
+    )
+    (property "Datasheet" "~" (at 85.09 57.15 0)
+      (effects (font (size 1.27 1.27)) hide)
+    )
+    (pin "1")
+    (pin "10")
+    (pin "11")
+    (pin "12")
+    (pin "2")
+    (pin "3")
+    (pin "4")
+    (pin "5")
+    (pin "6")
+    (pin "7")
+    (pin "8")
+    (pin "9")
+    (instances
+      (project "wii-pmod-adapter"
+        (path "/3e768cc3-1b06-47e6-92bc-2e81f82d9573"
+          (reference "J1") (unit 1)
+        )
+      )
+    )
+  )
   (symbol (lib_id "Device:D_Schottky") (at 163.83 30.48 180) (unit 1)
     (in_bom yes) (on_board yes) (dnp no)
@@
       (effects (font (size 1.27 1.27)) hide)
     )
-    (property "Footprint" "" (at 163.83 30.48 0)
+    (property "Footprint" "Diode_SMD:D_SOD-123" (at 163.83 30.48 0)
       (effects (font (size 1.27 1.27)) hide)
     )
@@
       (effects (font (size 1.27 1.27)) hide)
     )
-    (property "Footprint" "" (at 163.83 34.29 0)
+    (property "Footprint" "Diode_SMD:D_SOD-123" (at 163.83 34.29 0)
       (effects (font (size 1.27 1.27)) hide)
     )
@@
     )
   )
-  (symbol (lib_id "Connector_Generic:Conn_02x06_Row_Letter_First") (at 124.46 57.15 0) (unit 1)
+  (symbol (lib_id "Connector:Conn_01x02_Pin") (at 151.13 99.06 0) (unit 1)
+    (in_bom yes) (on_board yes) (dnp no) (fields_autoplaced)
+    (property "Reference" "J3" (at 151.765 93.98 0)
+      (effects (font (size 1.27 1.27)))
+    )
+    (property "Value" "PWR" (at 151.765 96.52 0)
+      (effects (font (size 1.27 1.27)))
+    )
+    (property "Footprint" "Connector_JST:JST_PH_B2B-PH-K_1x02_P2.00mm_Vertical" (at 151.13 99.06 0)
+      (effects (font (size 1.27 1.27)) hide)
+    )
+    (property "Datasheet" "~" (at 151.13 99.06 0)
+      (effects (font (size 1.27 1.27)) hide)
+    )
+    (pin "1")
+    (pin "2")
+    (instances
+      (project "wii-pmod-adapter"
+        (path "/3e768cc3-1b06-47e6-92bc-2e81f82d9573"
+          (reference "J3") (unit 1)
+        )
+      )
+    )
+  )
+  (symbol (lib_id "Connector_Generic:Conn_02x06_Odd_Even") (at 124.46 57.15 0) (unit 1)
     (in_bom yes) (on_board yes) (dnp no) (fields_autoplaced)
     (property "Reference" "J2" (at 125.73 45.72 0)
       (effects (font (size 1.27 1.27)))
     )
-    (property "Value" "PMOD1" (at 125.73 48.26 0)
-      (effects (font (size 1.27 1.27)))
-    )
-    (property "Footprint" "" (at 124.46 57.15 0)
+    (property "Value" "Conn_02x06_Odd_Even" (at 125.73 48.26 0)
+      (effects (font (size 1.27 1.27)))
+    )
+    (property "Footprint" "Connector_PinHeader_2.54mm:PinHeader_2x06_P2.54mm_Vertical" (at 124.46 57.15 0)
       (effects (font (size 1.27 1.27)) hide)
     )
@@
       (effects (font (size 1.27 1.27)) hide)
     )
-    (pin "a1")
-    (pin "a2")
-    (pin "a3")
-    (pin "a4")
-    (pin "a5")
-    (pin "a6")
-    (pin "b1")
-    (pin "b2")
-    (pin "b3")
-    (pin "b4")
-    (pin "b5")
-    (pin "b6")
+    (pin "1")
+    (pin "10")
+    (pin "11")
+    (pin "12")
+    (pin "2")
+    (pin "3")
+    (pin "4")
+    (pin "5")
+    (pin "6")
+    (pin "7")
+    (pin "8")
+    (pin "9")
     (instances
       (project "wii-pmod-adapter"
         (path "/3e768cc3-1b06-47e6-92bc-2e81f82d9573"
           (reference "J2") (unit 1)
-        )
-      )
-    )
-  )
-  (symbol (lib_id "Connector:Conn_01x02_Pin") (at 151.13 99.06 0) (unit 1)
-    (in_bom yes) (on_board yes) (dnp no) (fields_autoplaced)
-    (property "Reference" "J3" (at 151.765 93.98 0)
-      (effects (font (size 1.27 1.27)))
-    )
-    (property "Value" "PWR" (at 151.765 96.52 0)
-      (effects (font (size 1.27 1.27)))
-    )
-    (property "Footprint" "" (at 151.13 99.06 0)
-      (effects (font (size 1.27 1.27)) hide)
-    )
-    (property "Datasheet" "~" (at 151.13 99.06 0)
-      (effects (font (size 1.27 1.27)) hide)
-    )
-    (pin "1")
-    (pin "2")
-    (instances
-      (project "wii-pmod-adapter"
-        (path "/3e768cc3-1b06-47e6-92bc-2e81f82d9573"
-          (reference "J3") (unit 1)
         )
       )
@@
       (effects (font (size 1.27 1.27)) hide)
     )
-    (property "Footprint" "" (at 163.83 26.67 0)
+    (property "Footprint" "Diode_SMD:D_SOD-123" (at 163.83 26.67 0)
       (effects (font (size 1.27 1.27)) hide)
     )
@@
       (effects (font (size 1.27 1.27)) hide)
     )
-    (property "Footprint" "" (at 163.83 83.82 0)
+    (property "Footprint" "Diode_SMD:D_SOD-123" (at 163.83 83.82 0)
       (effects (font (size 1.27 1.27)) hide)
     )
@@
       (effects (font (size 1.27 1.27)) hide)
     )
-    (property "Footprint" "" (at 163.83 38.1 0)
+    (property "Footprint" "Diode_SMD:D_SOD-123" (at 163.83 38.1 0)
       (effects (font (size 1.27 1.27)) hide)
     )
@@
       (effects (font (size 1.27 1.27)) hide)
     )
-    (property "Footprint" "" (at 163.83 91.44 0)
+    (property "Footprint" "Diode_SMD:D_SOD-123" (at 163.83 91.44 0)
       (effects (font (size 1.27 1.27)) hide)
     )
@@
       (effects (font (size 1.27 1.27)) hide)
     )
-    (property "Footprint" "" (at 163.83 63.5 0)
+    (property "Footprint" "Diode_SMD:D_SOD-123" (at 163.83 63.5 0)
       (effects (font (size 1.27 1.27)) hide)
     )
@@
       (effects (font (size 1.27 1.27)) hide)
     )
-    (property "Footprint" "" (at 163.83 80.01 0)
-      (effects (font (size 1.27 1.27)) hide)
-    )
+    (property "Footprint" "Diode_SMD:D_SOD-123" (at 163.83 80.01 0)
+      (effects (font (size 1.27 1.27)) hide)
+    )
